File: scemetic.sch (KiCad schematic (older format))
At the start: 9 parts, among them J1 NRF24, J2 SPI connector, U1 ATTINY85-20PU

Commit message: receiver
Parts:
- removed BT1: Battery_Cell, symbol Battery_Cell
- removed D1: RED, symbol LED
- removed D2: GREEN, symbol LED
- added C?: 47 uF, symbol CP
- added J?: HIGH VOLTAGE LINE 01, symbol Conn_01x01_Female
- added J?: HIGH VOLTAGE LINE 02, symbol Conn_01x01_Female
- added J?: HIGH VOLTAGE GROUND, symbol Conn_01x01_Female
- added NE? (x2): Lamp_Neon, symbol Lamp_Neon
- added R? (x2): LDR03, Opto-Devices:Resistor_LDR_10x8.5_RM7.6, symbol LDR03
- added SC?: Solar_Cell, symbol Solar_Cell
Connections:
- net at C1.2, J1.1 (Pin_1), J1.10 (Pin_10)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: now also C?.2, R?.1, R?.1, SC?.2 (-)
- net at U1.3 (PB4(XTAL2/CLKO/OC1B/ADC2/PCINT4)): now also R?.2
- net at J2.6 (Pin_6), U1.5 (PB0(MOSI/DI/SDA/AIN0/OC0A/OC1A/AREF/PCINT0)): now also R?.2
- net at J1.5 (Pin_5), J1.6 (Pin_6), J2.5 (Pin_5): now also C?.1, SC?.1 (+)
- new net: J?.1 (Pin_1), NE?.1, NE?.1
- new net: J?.1 (Pin_1), NE?.2 (x2)
